File: KiCad files/Guitar Pedal.kicad_pcb (KiCad board)
At the start: 2 copper layers, 100.5 x 52 mm, 16 parts, among them CN1 Guitar Input, CN2 Guitar Output, U1 Op-Amp, U2 LiPo Charger, U3 I2S DAC

Commit message: Drill holes, 3D KiCad outputs
Parts:
- added REF**: MountingHole_2.2mm_M2, MountingHole:MountingHole_2.2mm_M2, F.Cu at (158.5, 90.0)
- added REF**: MountingHole_2.2mm_M2, MountingHole:MountingHole_2.2mm_M2, F.Cu at (189.0, 99.0)
- added REF**: MountingHole_2.2mm_M2, MountingHole:MountingHole_2.2mm_M2, F.Cu at (117.0, 99.5)
